File: KiCad/c264-magic-cart-rev1.kicad_sch (KiCad schematic)
At the start: 10 parts, among them IC1 27C080, IC2 74LS/HCT273, IC3 27C160, IC5 GAL20V8

Commit message: Some rought edges, but ready for V1S
Parts:
- removed C2, C3: C-EU025-024X044, c264-magic-cart-rev1:C025-024X044, symbol c264-magic-cart-rev1-eagle-import:C-EU025-024X044
- removed IC1: 27C080, c264-magic-cart-rev1:DIL32, symbol c264-magic-cart-rev1-eagle-import:27C08032P6
- removed IC2: 74LS/HCT273, c264-magic-cart-rev1:DIL20, symbol c264-magic-cart-rev1-eagle-import:74273N
- removed IC5: GAL20V8, c264-magic-cart-rev1:DIL24-3, symbol c264-magic-cart-rev1-eagle-import:20V8
- removed U$1: C16_CARTRIDGE, c264-magic-cart-rev1:C16_CART, symbol c264-magic-cart-rev1-eagle-import:C16_CARTRIDGE
- added C2, C3: 100n, Capacitor_THT:C_Disc_D7.5mm_W2.5mm_P5.00mm, symbol Device:C
- added CN1: C16_NEWSTYLE_EXP_PORT, c264-magic-cart-rev1:EdgeConn-44pin, symbol C16-Exp-Port-44pin-In:C16_NEWSTYLE_EXP_PORT
- added U1: 27C080, Package_DIP:DIP-32_W15.24mm_Socket, symbol Memory_EPROM:27C080
- added U2: 74HCT273, Package_DIP:DIP-20_W7.62mm_Socket_LongPads, symbol 74xx:74HCT273
- added U5: GAL20V8, Package_DIP:DIP-24_W7.62mm_Socket_LongPads, symbol Logic_Programmable:PAL20L8
- U3: renamed from IC3; footprint c264-magic-cart-rev1:DIP42 -> Package_DIP:DIP-42_W15.24mm_Socket
Connections:
- net /CRT: now also U2.11 (Cp), U5.15 (IO15)
- net /RESET: now also CN1.C (~{RESET}), U2.1 (~{Mr})
- net A0: now also CN1.Y (A0), U1.12 (A0), U5.10 (I10)
- net A1: now also CN1.X (A1), U1.11 (A1), U5.19 (IO19)
- net A10: now also CN1.M (A10), U1.23 (A10), U5.5 (I5)
- net A11: now also CN1.L (A11), U1.25 (A11), U5.23 (I23)
- net A12: now also CN1.K (A12), U1.4 (A12), U5.16 (IO16)
- net A13: now also CN1.J (A13), U1.28 (A13), U5.21 (IO21)
- net A14: now also CN1.H (A14), U5.3 (I3)
- net A15: now also CN1.F (A15), U5.2 (I2)
- net A2: now also CN1.W (A2), U1.10 (A2), U5.7 (I7)
- net A3: now also CN1.V (A3), U1.9 (A3), U5.20 (I020)
- net A4: now also CN1.U (A4), U1.8 (A4), U5.8 (I8)
- net A5: now also CN1.T (A5), U1.7 (A5), U5.18 (IO18)
- net A6: now also CN1.S (A6), U1.6 (A6), U5.9 (I9)
- net A7: now also CN1.R (A7), U1.5 (A7), U5.17 (IO17)
- net A8: now also CN1.P (A8), U1.27 (A8), U5.6 (I6)
- net A9: now also CN1.N (A9), U1.26 (A9), U5.4 (I4)
- net AA14: now also U1.29 (A14), U2.12 (Q4)
- net AA15: now also U1.3 (A15), U2.15 (Q5)
- net AA16: now also U1.2 (A16), U2.6 (Q2)
- net AA17: now also U1.30 (A17), U2.9 (Q3)
- net AA18: now also U2.2 (Q0)
- net AA19: now also U2.5 (Q1)
- net AA20: now also U2.16 (Q6)
- net AA21: now also U2.19 (Q7)
- net C1LO: now also CN1.B (~{C1LO}), U1.22 (~{CE}), U1.24 (~{OE})
- net CFG0: now also U5.13 (I13)
- net CFG1: now also U5.14 (I14)
- net D0: now also CN1.21 (D0), U1.13 (D0), U2.13 (D4)
- net D1: now also CN1.20 (D1), U1.14 (D1), U2.14 (D5)
- net D2: now also CN1.19 (D2), U1.15 (D2), U2.7 (D2)
- net D3: now also CN1.18 (D3), U1.17 (D3), U2.8 (D3)
- net D4: now also CN1.17 (D4), U1.18 (D4), U2.3 (D0)
- net D5: now also CN1.16 (D5), U1.19 (D5), U2.4 (D1)
- net D6: now also CN1.15 (D6), U1.20 (D6), U2.17 (D6)
- net D7: now also CN1.14 (D7), U1.21 (D7), U2.18 (D7)
- net GND: now also C2.2, C3.2, CN1.1 (GND), CN1.22 (GND), CN1.A (GND), CN1.Z (GND), U1.16 (GND), U2.10 (GND), U5.12 (GND)
- net PHI2: now also CN1.6 (PHI2), U5.11 (I11)
- net PIN1: now also U1.1 (A19)
- net PIN31: now also U1.31 (A18)
- net R/W: now also CN1.5 (R/~{W}), U5.1 (I1)
- net VCC: now also C2.1, C3.1, CN1.2 (+5V), CN1.3 (+5V), U1.32 (VCC), U2.20 (VCC), U5.24 (VCC)
- no-connect marks 0 -> 11
Other:
- moved on the sheet: CONFIG0
